File: hardware/hip9011/DD HIP9011.sch (KiCad schematic (older format))
At the start: 34 parts, among them P1 KNOCK 1, P2 KNOCK 2, P3 12V, P4 CONN_5X2, P5 CONN_2, P6 CONN_2, U1 7805-SOT89, X1 QUARTZ

Commit message: new version
Parts:
- added G1: LOGO, symbol LOGO
Changed lines of the file:
@@
 LIBS:quartz
 LIBS:7805-sot89
+LIBS:logo_flipped
 LIBS:DD HIP9011-cache
 EELAYER 27 0
@@
 Text Label 8350 5950 0    60   ~ 0
 GND
+$Comp
+L LOGO G1
+U 1 1 52AF4640
+P 3950 2700
+F 0 "G1" H 3950 2597 60  0001 C CNN
+F 1 "LOGO" H 3950 2803 60  0001 C CNN
+F 2 "" H 3950 2700 60  0000 C CNN
+F 3 "" H 3950 2700 60  0000 C CNN
+	1    3950 2700
+	1    0    0    -1
+$EndComp
 $EndSCHEMATC
