File: hardware/adc_amp_divider.vertical/adc_amp_divider.kicad_pcb (KiCad board)
At the start: 2 copper layers, 47 x 70 mm, 83 parts, among them M200 CONN_1, M201 CONN_1, M202 CONN_1, P201 CONN_10X2, P202 CONN_3, P203 CONN_2, P204 CONN_1, P205 CONN_1, P208 CONN_6, P209 CONN_6, U201 LMV324IDR, U202 LMV324IDR

Commit message: vertical version - clean-up
Parts:
- removed P209: CONN_6, PIN_ARRAY-6X1
- added P207: CONN_2, PIN_ARRAY_2X1, F.Cu at (145.4, 95.9)
- moved M200 160.5 mm to (170.6, 136.1)
- moved G201 122.6 mm to (168.3, 109.5)
- moved M201 105.6 mm to (170.7, 161.4)
- moved P205 49.6 mm to (133.2, 135.5)
- moved M202 20.6 mm to (128.7, 102.5)
- moved P204 20.1 mm to (133.5, 144.8)
- moved P202 4.51 mm to (158.8, 96.0)
- moved P208 1.17 mm to (134.2, 95.9)
- moved P203 0.57 mm to (169.5, 96.0)
Routing:
- net VCC: track 384.5 -> 193.3 mm, vias 6 -> 4
- net /INP7: track 56.3 -> 14.1 mm
- net /OUT7: track 35.1 -> 3.17 mm
- net /OUT8: track 29.0 -> 3.43 mm
- net /OUT5: track 25.5 -> 3.17 mm
- net /OUT3: track 22.7 -> 3.17 mm
- net /OUT6: track 22.4 -> 3.43 mm
- net /OUT4: track 20.7 -> 3.17 mm
- net /INP6: track 33.0 -> 16.2 mm
- net /OUT1: track 19.5 -> 3.17 mm
- net (no net): track 16.2 -> 0.25 mm
- net /INP4: track 31.1 -> 16.2 mm
- net /OUT2: track 15.2 -> 3.17 mm
- net /INP3: track 25.4 -> 13.4 mm
- net /INP2: track 26.9 -> 15.3 mm
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
Commit message: improved version
Parts:
- added P209: CONN_1, PIN_ARRAY_1, F.Cu at (135.9, 142.6)
- moved M201 61.0 mm to (167.9, 100.5)
- moved LD200 55.6 mm to (128.4, 108.5), turned to 270 degrees
- moved R200 47.4 mm to (128.4, 115.3), turned to 90 degrees
- moved G201 16.0 mm to (152.4, 111.6)
- moved M200 8.61 mm to (167.4, 144.1)
- moved P203 5.46 mm to (164.1, 95.9)
- moved P202 3.94 mm to (154.8, 95.9)
- moved P204 1.14 mm to (133.0, 145.8)
- moved P205 0.90 mm to (133.9, 136.1)
Connections:
- P201 pad 12: (no net) -> /OUT7
- P201 pad 14: /OUT7 -> /OUT5
- P201 pad 16: /OUT5 -> /PA4
Routing:
- net GND: track 64.9 -> 59.3 mm, vias 36 -> 32
- net N-0000011: track 2.55 -> 0.00 mm
- net VCC: track 193.3 -> 191.7 mm
Other:
- board size 47 x 70 mm -> 44 x 70 mm

Commit message: now with bad tracks
Routing:
- net /OUT8: track 3.43 -> 48.7 mm, vias 0 -> 1
- net VCC: track 191.7 -> 235.8 mm
- net /OUT7: track 3.17 -> 40.3 mm, vias 0 -> 1
- net /OUT6: track 3.43 -> 39.7 mm, vias 0 -> 1
- net /OUT4: track 3.17 -> 32.2 mm
- net /OUT5: track 3.17 -> 30.9 mm, vias 0 -> 1
- net /INP8: track 15.3 -> 39.3 mm
- net /OUT3: track 3.17 -> 22.6 mm, vias 0 -> 1
- net /INP6: track 16.2 -> 35.5 mm
- net /INP7: track 14.1 -> 31.7 mm
- net /INP4: track 16.2 -> 31.9 mm
- net /OUT1: track 3.17 -> 17.8 mm
- net /OUT2: track 3.17 -> 17.7 mm
- net /INP5: track 15.9 -> 29.8 mm
- net /INP3: track 13.4 -> 25.7 mm
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- added copper zone on F.Cu, net GND
- removed copper zone on F.Cu, net VCC
Other:
- net class Default: clearance 0.2032 -> 0.0254
- rule trace_clearance: 0.2032 -> 0.0254

Commit message: better version
Routing:
- net N-0000026: track 20.7 -> 21.4 mm
Other:
- net class Default: clearance 0.0254 -> 0.2032
- rule trace_clearance: 0.0254 -> 0.2032
Changed lines of the file:
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@@
     (18 B.Paste user)
     (19 F.Paste user)
-    (20 B.SilkS user)
-    (21 F.SilkS user)
+    (20 B.SilkS user hide)
+    (21 F.SilkS user hide)
     (22 B.Mask user)
     (23 F.Mask user)
@@
   (setup
     (last_trace_width 0.254)
-    (trace_clearance 0.0254)
+    (trace_clearance 0.2032)
     (zone_clearance 0.254)
     (zone_45_only no)
@@
   (net 46 VCC)
   (net_class Default "This is the default net class."
-    (clearance 0.0254)
+    (clearance 0.2032)
     (trace_width 0.254)
     (via_dia 0.889)
@@
   (segment (start 147.955 131.064) (end 147.955 127.889) (width 0.254) (layer F.Cu) (net 29))
   (segment (start 147.981 131.09) (end 147.955 131.064) (width 0.254) (layer F.Cu) (net 29))
-  (segment (start 147.981 141.296) (end 147.981 131.09) (width 0.254) (layer F.Cu) (net 29))
-  (segment (start 146.148 143.129) (end 147.981 141.296) (width 0.254) (layer F.Cu) (net 29))
+  (segment (start 148.59 141.224) (end 147.981 131.09) (width 0.254) (layer F.Cu) (net 29))
+  (segment (start 146.148 143.129) (end 148.59 141.224) (width 0.254) (layer F.Cu) (net 29))
   (segment (start 145.923 143.129) (end 146.148 143.129) (width 0.254) (layer F.Cu) (net 29))
   (segment (start 165.1 127.889) (end 165.1 131.064) (width 0.254) (layer F.Cu) (net 30))
@@
   (segment (start 146.438 154.679) (end 145.288 155.829) (width 0.254) (layer F.Cu) (net 32))
   (segment (start 146.438 148.088) (end 146.438 154.679) (width 0.254) (layer F.Cu) (net 32))
-  (segment (start 145.543 147.193) (end 146.438 148.088) (width 0.254) (layer F.Cu) (net 32))
-  (segment (start 144.653 147.193) (end 145.543 147.193) (width 0.254) (layer F.Cu) (net 32))
-  (segment (start 144.016 146.556) (end 144.653 147.193) (width 0.254) (layer F.Cu) (net 32))
-  (segment (start 144.016 141.004) (end 144.016 146.556) (width 0.254) (layer F.Cu) (net 32))
-  (segment (start 145.701 139.319) (end 144.016 141.004) (width 0.254) (layer F.Cu) (net 32))
+  (segment (start 145.543 147.447) (end 146.438 148.088) (width 0.254) (layer F.Cu) (net 32))
+  (segment (start 144.399 147.447) (end 145.543 147.447) (width 0.254) (layer F.Cu) (net 32))
+  (segment (start 143.637 146.558) (end 144.399 147.447) (width 0.254) (layer F.Cu) (net 32))
+  (segment (start 143.637 140.97) (end 143.637 146.558) (width 0.254) (layer F.Cu) (net 32))
+  (segment (start 145.701 139.319) (end 143.637 140.97) (width 0.254) (layer F.Cu) (net 32))
   (segment (start 145.923 139.319) (end 145.701 139.319) (width 0.254) (layer F.Cu) (net 32))
   (segment (start 154.686 132.588) (end 156.21 131.064) (width 0.254) (layer F.Cu) (net 33))
@@
   (segment (start 150.431 119.317) (end 149.733 120.015) (width 0.254) (layer F.Cu) (net 46))
   (segment (start 150.962 119.317) (end 150.431 119.317) (width 0.254) (layer F.Cu) (net 46))
-  (segment (start 145.604 135.509) (end 147.473 137.378) (width 0.254) (layer F.Cu) (net 46))
+  (segment (start 145.604 135.509) (end 147.574 136.652) (width 0.254) (layer F.Cu) (net 46))
   (segment (start 144.082 135.509) (end 145.604 135.509) (width 0.254) (layer F.Cu) (net 46))
   (segment (start 158.242 130.937) (end 160.02 132.715) (width 0.254) (layer B.Cu) (net 46))
@@
   (segment (start 142.557 115.507) (end 141.224 116.84) (width 0.254) (layer F.Cu) (net 46))
   (segment (start 142.632 115.507) (end 142.557 115.507) (width 0.254) (layer F.Cu) (net 46))
-  (segment (start 147.473 140.554) (end 147.473 137.378) (width 0.254) (layer F.Cu) (net 46))
-  (segment (start 146.168 141.859) (end 147.473 140.554) (width 0.254) (layer F.Cu) (net 46))
+  (segment (start 147.701 140.589) (end 147.574 136.652) (width 0.254) (layer F.Cu) (net 46))
+  (segment (start 146.168 141.859) (end 147.701 140.589) (width 0.254) (layer F.Cu) (net 46))
   (segment (start 145.923 141.859) (end 146.168 141.859) (width 0.254) (layer F.Cu) (net 46))
-  (segment (start 147.473 137.378) (end 145.605 135.509) (width 0.254) (layer F.Cu) (net 46))
+  (segment (start 147.574 136.652) (end 145.605 135.509) (width 0.254) (layer F.Cu) (net 46))
   (segment (start 159.957 135.509) (end 160.02 135.446) (width 0.254) (layer F.Cu) (net 46))
   (segment (start 159.9565 135.509) (end 159.957 135.509) (width 0.254) (layer F.Cu) (net 46))
