File: hardware/1A_injector_6-channels/inj_6ch.sch (KiCad schematic (older format))
At the start: 29 parts, among them P1 CONN_10X2, P2 CONN_2, P3 CONN_3, P4 CONN_2, P5 CONN_3, P7 CONN_10X2, Q1 OVP_DRIVER, Q2 OVP_DRIVER, Q3 OVP_DRIVER, Q4 OVP_DRIVER, Q5 OVP_DRIVER, Q6 OVP_DRIVER

Commit message: 
Parts:
- added R4, R5, R6, R7, R8, R9: 20R, SM0805, symbol R
Changed lines of the file:
@@
 Sheet 1 1
 Title "6 Channel Injector"
-Date "10 nov 2013"
-Rev "A-5"
+Date "1 dec 2013"
+Rev "A-6"
 Comp "http://code.google.com/p/daecu/"
 Comment1 ""
@@
 	3900 3525 3950 3525
 Connection ~ 3900 2225
-Wire Wire Line
-	3900 2125 4450 2125
 Wire Wire Line
 	3900 2125 3900 2275
@@
 Text Label 4875 2375 0    60   ~ 0
 iGND1
-Text Label 3900 2725 2    60   ~ 0
+Text Label 3450 2725 2    60   ~ 0
 INJ-05_5V
-Text Label 4425 2125 2    60   ~ 0
+Text Label 3400 2225 2    60   ~ 0
 INJ-06_5V
 $Comp
@@
 Text Label 4900 3625 0    60   ~ 0
 iGND1
-Text Label 3900 3975 2    60   ~ 0
+Text Label 3450 3975 2    60   ~ 0
 INJ-03_5V
-Text Label 4425 3375 2    60   ~ 0
+Text Label 3400 3475 2    60   ~ 0
 INJ-04_5V
 $Comp
@@
 	0    1    1    0
 $EndComp
-Text Label 4425 4625 2    60   ~ 0
+Text Label 3400 4725 2    60   ~ 0
 INJ-02_5V
-Text Label 3900 5225 2    60   ~ 0
+Text Label 3450 5225 2    60   ~ 0
 INJ-01_5V
 Text Label 4875 4875 0    60   ~ 0
@@
 Text Label 5400 2375 3    60   ~ 0
 INJ-06_2
+$Comp
+L R R4
+U 1 1 529A8640
+P 3650 2225
+F 0 "R4" V 3730 2225 50  0000 C CNN
+F 1 "20R" V 3650 2225 50  0000 C CNN
+F 2 "SM0805" V 580 -150 60  0001 C CNN
+F 3 "" H 3650 2225 60  0001 C CNN
+F 4 "Panasonic,ECG ERJ-6ENF20R0V" V 580 -150 60  0001 C CNN "mfg,mfg#"
+F 5 "digi,ERJ-6ENF20R0V" V 580 -150 60  0001 C CNN "vend1,vend1#"
+	1    3650 2225
+	0    1    1    0
+$EndComp
+Wire Wire Line
+	3900 2125 4450 2125
+$Comp
+L R R7
+U 1 1 529A8879
+P 3700 2725
+F 0 "R7" V 3780 2725 50  0000 C CNN
+F 1 "20R" V 3700 2725 50  0000 C CNN
+F 2 "SM0805" V 630 350 60  0001 C CNN
+F 3 "" H 3700 2725 60  0001 C CNN
+F 4 "Panasonic,ECG ERJ-6ENF20R0V" V 630 350 60  0001 C CNN "mfg,mfg#"
+F 5 "digi,ERJ-6ENF20R0V" V 630 350 60  0001 C CNN "vend1,vend1#"
+	1    3700 2725
+	0    1    1    0
+$EndComp
+$Comp
+L R R5
+U 1 1 529A8883
+P 3650 3475
+F 0 "R5" V 3730 3475 50  0000 C CNN
+F 1 "20R" V 3650 3475 50  0000 C CNN
+F 2 "SM0805" V 580 1100 60  0001 C CNN
+F 3 "" H 3650 3475 60  0001 C CNN
+F 4 "Panasonic,ECG ERJ-6ENF20R0V" V 580 1100 60  0001 C CNN "mfg,mfg#"
+F 5 "digi,ERJ-6ENF20R0V" V 580 1100 60  0001 C CNN "vend1,vend1#"
+	1    3650 3475
+	0    1    1    0
+$EndComp
+$Comp
+L R R8
+U 1 1 529A888D
+P 3700 3975
+F 0 "R8" V 3780 3975 50  0000 C CNN
+F 1 "20R" V 3700 3975 50  0000 C CNN
+F 2 "SM0805" V 630 1600 60  0001 C CNN
+F 3 "" H 3700 3975 60  0001 C CNN
+F 4 "Panasonic,ECG ERJ-6ENF20R0V" V 630 1600 60  0001 C CNN "mfg,mfg#"
+F 5 "digi,ERJ-6ENF20R0V" V 630 1600 60  0001 C CNN "vend1,vend1#"
+	1    3700 3975
+	0    1    1    0
+$EndComp
+$Comp
+L R R6
+U 1 1 529A8899
+P 3650 4725
+F 0 "R6" V 3730 4725 50  0000 C CNN
+F 1 "20R" V 3650 4725 50  0000 C CNN
+F 2 "SM0805" V 580 2350 60  0001 C CNN
+F 3 "" H 3650 4725 60  0001 C CNN
+F 4 "Panasonic,ECG ERJ-6ENF20R0V" V 580 2350 60  0001 C CNN "mfg,mfg#"
+F 5 "digi,ERJ-6ENF20R0V" V 580 2350 60  0001 C CNN "vend1,vend1#"
+	1    3650 4725
+	0    1    1    0
+$EndComp
+$Comp
+L R R9
+U 1 1 529A88A3
+P 3700 5225
+F 0 "R9" V 3780 5225 50  0000 C CNN
+F 1 "20R" V 3700 5225 50  0000 C CNN
+F 2 "SM0805" V 630 2850 60  0001 C CNN
+F 3 "" H 3700 5225 60  0001 C CNN
+F 4 "Panasonic,ECG ERJ-6ENF20R0V" V 630 2850 60  0001 C CNN "mfg,mfg#"
+F 5 "digi,ERJ-6ENF20R0V" V 630 2850 60  0001 C CNN "vend1,vend1#"
+	1    3700 5225
+	0    1    1    0
+$EndComp
 $EndSCHEMATC

Commit message: working with BOM
Parts:
- removed P1, P7: CONN_10X2, pin_array_10x2, symbol CONN_10X2
- added P1, P7: HEADER_10X2, ~, symbol HEADER_10X2
Changed lines of the file:
@@
 EESchema Schematic File Version 2
 LIBS:project_specific_libs
+LIBS:header_10x2
 LIBS:power
 LIBS:device
@@
 Sheet 1 1
 Title "6 Channel Injector"
-Date "1 dec 2013"
+Date "24 dec 2013"
 Rev "A-6"
 Comp "http://code.google.com/p/daecu/"
@@
 Wire Notes Line
 	9350 3425 8025 3425
-$Comp
-L CONN_10X2 P1
-U 1 1 527CB514
-P 1675 6825
-F 0 "P1" H 1675 7375 60  0000 C CNN
-F 1 "CONN_10X2" V 1675 6725 50  0000 C CNN
-F 2 "pin_array_10x2" H 1675 6825 60  0001 C CNN
-F 3 "" H 1675 6825 60  0000 C CNN
-	1    1675 6825
-	1    0    0    -1
-$EndComp
 $Comp
 L CONN_3 P3
@@
 Wire Wire Line
 	1075 6375 1275 6375
-$Comp
-L CONN_10X2 P7
-U 1 1 527E2500
-P 2975 6825
-F 0 "P7" H 2975 7375 60  0000 C CNN
-F 1 "CONN_10X2" V 2975 6800 50  0000 C CNN
-F 2 "pin_array_10x2" H 2975 6825 60  0001 C CNN
-F 3 "" H 2975 6825 60  0000 C CNN
-	1    2975 6825
-	1    0    0    -1
-$EndComp
 Wire Wire Line
 	2075 6375 2575 6375
@@
 	0    1    1    0
 $EndComp
+$Comp
+L HEADER_10X2 P1
+U 1 1 52B99314
+P 1675 6825
+F 0 "P1" H 1675 7375 60  0000 C CNN
+F 1 "HEADER_10X2" V 1675 6725 50  0000 C CNN
+F 2 "~" H 1675 6825 60  0000 C CNN
+F 3 "~" H 1675 6825 60  0000 C CNN
+F 4 "TE,1-215307-0" H 1775 7475 60  0000 C CNN "mfg,mfg#"
+F 5 "digi,A106616-ND" H 1875 7575 60  0000 C CNN "vend1,vend1#"
+	1    1675 6825
+	1    0    0    -1
+$EndComp
+$Comp
+L HEADER_10X2 P7
+U 1 1 52B99443
+P 2975 6825
+F 0 "P7" H 2975 7375 60  0000 C CNN
+F 1 "HEADER_10X2" V 2975 6725 50  0000 C CNN
+F 2 "~" H 2975 6825 60  0000 C CNN
+F 3 "~" H 2975 6825 60  0000 C CNN
+F 4 "TE,1-215307-0" H 3075 7475 60  0000 C CNN "mfg,mfg#"
+F 5 "digi,A106616-ND" H 3175 7575 60  0000 C CNN "vend1,vend1#"
+	1    2975 6825
+	1    0    0    -1
+$EndComp
 $EndSCHEMATC
