File: trunk/hardware/frankenstein_foundation/frankenstein_foundation.kicad_pcb (KiCad board)
At the start: 2 copper layers, 100 x 99.9 mm, 7 parts, among them P1 CONN_4X2, P2 CONN_10X2, P3 CONN_2, P4 CONN_5X2

Commit message: nicer module
Parts:
- P2: footprint PIN_ARRAY_10X2 -> PIN_ARRAY_10X2_M
Changed lines of the file:
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@@
-    )
-  )
-  (module PIN_ARRAY_10X2 (layer F.Cu)
-    (at 128.27 176.53 270)
-    (descr "Double rangee de contacts 2 x 10 pins")
-    (tags CONN)
-    (fp_text reference P2 (at 0 -3.81 270) (layer F.SilkS)
-      (effects (font (size 1.016 1.016) (thickness 0.254)))
-    )
-    (fp_text value CONN_10X2 (at 0 3.81 270) (layer F.SilkS)
-      (effects (font (size 1.016 1.016) (thickness 0.2032)))
-    )
-    (fp_line (start 12.7 2.54) (end -12.7 2.54) (layer F.SilkS) (width 0.381))
-    (fp_line (start -12.7 -2.54) (end 12.7 -2.54) (layer F.SilkS) (width 0.381))
-    (fp_line (start -12.7 -2.54) (end -12.7 2.54) (layer F.SilkS) (width 0.381))
-    (fp_line (start 12.7 2.54) (end 12.7 -2.54) (layer F.SilkS) (width 0.381))
-    (pad 1 thru_hole rect (at -11.43 1.27 270) (size 1.524 1.524) (drill 0.8128)
-      (layers *.Cu *.Mask F.SilkS)
-    )
-    (pad 2 thru_hole circle (at -11.43 -1.27 270) (size 1.524 1.524) (drill 1.016)
-      (layers *.Cu *.Mask F.SilkS)
-    )
-    (pad 3 thru_hole circle (at -8.89 1.27 270) (size 1.524 1.524) (drill 1.016)
-      (layers *.Cu *.Mask F.SilkS)
-    )
-    (pad 4 thru_hole circle (at -8.89 -1.27 270) (size 1.524 1.524) (drill 1.016)
-      (layers *.Cu *.Mask F.SilkS)
-    )
-    (pad 5 thru_hole circle (at -6.35 1.27 270) (size 1.524 1.524) (drill 1.016)
-      (layers *.Cu *.Mask F.SilkS)
-    )
-    (pad 6 thru_hole circle (at -6.35 -1.27 270) (size 1.524 1.524) (drill 1.016)
-      (layers *.Cu *.Mask F.SilkS)
-      (net 3 CAN_RX)
-    )
-    (pad 7 thru_hole circle (at -3.81 1.27 270) (size 1.524 1.524) (drill 1.016)
-      (layers *.Cu *.Mask F.SilkS)
-    )
-    (pad 8 thru_hole circle (at -3.81 -1.27 270) (size 1.524 1.524) (drill 1.016)
-      (layers *.Cu *.Mask F.SilkS)
-    )
-    (pad 9 thru_hole circle (at -1.27 1.27 270) (size 1.524 1.524) (drill 1.016)
-      (layers *.Cu *.Mask F.SilkS)
-    )
-    (pad 10 thru_hole circle (at -1.27 -1.27 270) (size 1.524 1.524) (drill 1.016)
-      (layers *.Cu *.Mask F.SilkS)
-    )
-    (pad 11 thru_hole circle (at 1.27 1.27 270) (size 1.524 1.524) (drill 1.016)
-      (layers *.Cu *.Mask F.SilkS)
-    )
-    (pad 12 thru_hole circle (at 1.27 -1.27 270) (size 1.524 1.524) (drill 1.016)
-      (layers *.Cu *.Mask F.SilkS)
-    )
-    (pad 13 thru_hole circle (at 3.81 1.27 270) (size 1.524 1.524) (drill 1.016)
-      (layers *.Cu *.Mask F.SilkS)
-    )
-    (pad 14 thru_hole circle (at 3.81 -1.27 270) (size 1.524 1.524) (drill 1.016)
-      (layers *.Cu *.Mask F.SilkS)
-    )
-    (pad 15 thru_hole circle (at 6.35 1.27 270) (size 1.524 1.524) (drill 1.016)
-      (layers *.Cu *.Mask F.SilkS)
-    )
-    (pad 16 thru_hole circle (at 6.35 -1.27 270) (size 1.524 1.524) (drill 1.016)
-      (layers *.Cu *.Mask F.SilkS)
-    )
-    (pad 17 thru_hole circle (at 8.89 1.27 270) (size 1.524 1.524) (drill 1.016)
-      (layers *.Cu *.Mask F.SilkS)
-    )
-    (pad 18 thru_hole circle (at 8.89 -1.27 270) (size 1.524 1.524) (drill 1.016)
-      (layers *.Cu *.Mask F.SilkS)
-    )
-    (pad 19 thru_hole circle (at 11.43 1.27 270) (size 1.524 1.524) (drill 1.016)
-      (layers *.Cu *.Mask F.SilkS)
-      (net 4 GND)
-    )
-    (pad 20 thru_hole circle (at 11.43 -1.27 270) (size 1.524 1.524) (drill 1.016)
-      (layers *.Cu *.Mask F.SilkS)
-      (net 4 GND)
-    )
-    (model pin_array/pins_array_12x2.wrl
-      (at (xyz 0 0 0))
-      (scale (xyz 1 1 1))
-      (rotate (xyz 0 0 0))
     )
   )
@@
     )
   )
+  (module PIN_ARRAY_10X2_M (layer F.Cu)
+    (at 128.27 176.53 270)
+    (fp_text reference P2 (at 0 -3.81 270) (layer F.SilkS)
+      (effects (font (size 1.016 1.016) (thickness 0.254)))
+    )
+    (fp_text value CONN_10X2 (at 0 3.81 270) (layer F.SilkS)
+      (effects (font (size 1.016 1.016) (thickness 0.2032)))
+    )
+    (fp_line (start 12.49934 2.49936) (end 12.49934 -2.49936) (layer F.SilkS) (width 0.09906))
+    (fp_line (start 12.49934 -2.49936) (end -12.7508 -2.49936) (layer F.SilkS) (width 0.09906))
+    (fp_line (start -12.7508 -2.49936) (end -12.7508 2.49936) (layer F.SilkS) (width 0.09906))
+    (fp_line (start -12.7508 2.49936) (end 12.49934 2.49936) (layer F.SilkS) (width 0.09906))
+    (pad 1 thru_hole rect (at -11.47064 1.27 270) (size 1.524 1.524) (drill 0.8128)
+      (layers *.Cu *.Mask F.SilkS)
+    )
+    (pad 2 thru_hole circle (at -11.47064 -1.27 270) (size 1.524 1.524) (drill 1.016)
+      (layers *.Cu *.Mask F.SilkS)
+    )
+    (pad 3 thru_hole circle (at -8.93064 1.27 270) (size 1.524 1.524) (drill 1.016)
+      (layers *.Cu *.Mask F.SilkS)
+    )
+    (pad 4 thru_hole circle (at -8.93064 -1.27 270) (size 1.524 1.524) (drill 1.016)
+      (layers *.Cu *.Mask F.SilkS)
+    )
+    (pad 5 thru_hole circle (at -6.39064 1.27 270) (size 1.524 1.524) (drill 1.016)
+      (layers *.Cu *.Mask F.SilkS)
+    )
+    (pad 6 thru_hole circle (at -6.39064 -1.27 270) (size 1.524 1.524) (drill 1.016)
+      (layers *.Cu *.Mask F.SilkS)
+      (net 3 CAN_RX)
+    )
+    (pad 7 thru_hole circle (at -3.85064 1.27 270) (size 1.524 1.524) (drill 1.016)
+      (layers *.Cu *.Mask F.SilkS)
+    )
+    (pad 8 thru_hole circle (at -3.85064 -1.27 270) (size 1.524 1.524) (drill 1.016)
+      (layers *.Cu *.Mask F.SilkS)
+    )
+    (pad 9 thru_hole circle (at -1.31064 1.27 270) (size 1.524 1.524) (drill 1.016)
+      (layers *.Cu *.Mask F.SilkS)
+    )
+    (pad 10 thru_hole circle (at -1.31064 -1.27 270) (size 1.524 1.524) (drill 1.016)
+      (layers *.Cu *.Mask F.SilkS)
+    )
+    (pad 11 thru_hole circle (at 1.22936 1.27 270) (size 1.524 1.524) (drill 1.016)
+      (layers *.Cu *.Mask F.SilkS)
+    )
+    (pad 12 thru_hole circle (at 1.22936 -1.27 270) (size 1.524 1.524) (drill 1.016)
+      (layers *.Cu *.Mask F.SilkS)
+    )
+    (pad 13 thru_hole circle (at 3.76936 1.27 270) (size 1.524 1.524) (drill 1.016)
+      (layers *.Cu *.Mask F.SilkS)
+    )
+    (pad 14 thru_hole circle (at 3.76936 -1.27 270) (size 1.524 1.524) (drill 1.016)
+      (layers *.Cu *.Mask F.SilkS)
+    )
+    (pad 15 thru_hole circle (at 6.30936 1.27 270) (size 1.524 1.524) (drill 1.016)
+      (layers *.Cu *.Mask F.SilkS)
+    )
+    (pad 16 thru_hole circle (at 6.30936 -1.27 270) (size 1.524 1.524) (drill 1.016)
+      (layers *.Cu *.Mask F.SilkS)
+    )
+    (pad 17 thru_hole circle (at 8.84936 1.27 270) (size 1.524 1.524) (drill 1.016)
+      (layers *.Cu *.Mask F.SilkS)
+    )
+    (pad 18 thru_hole circle (at 8.84936 -1.27 270) (size 1.524 1.524) (drill 1.016)
+      (layers *.Cu *.Mask F.SilkS)
+    )
+    (pad 19 thru_hole circle (at 11.38936 1.27 270) (size 1.524 1.524) (drill 1.016)
+      (layers *.Cu *.Mask F.SilkS)
+      (net 4 GND)
+    )
+    (pad 20 thru_hole circle (at 11.38936 -1.27 270) (size 1.524 1.524) (drill 1.016)
+      (layers *.Cu *.Mask F.SilkS)
+      (net 4 GND)
+    )
+    (model lib/3d/M_header_10x2.wrl
+      (at (xyz 0 0 0))
+      (scale (xyz 1 1 1))
+      (rotate (xyz -90 0 0))
+    )
+  )

Commit message: making progress
Parts:
- removed W1, W2, W3: TEST, SIL-2
- added JP1: JUMPER, SIL-2, F.Cu at (173.5, 180.3)
- added JP2: JUMPER, SIL-2, F.Cu at (171.2, 185.4)
- added JP3: JUMPER, SIL-2, F.Cu at (135.6, 170.2)
- renumbered P1 to P51, P2 to P52, P3 to P53, P4 to P54
Connections:
- P51 pad 1: /PA8 -> /CRANK
- P51 pad 5: /PC6 -> /CAM
Routing:
- net (no net): track 0.00 -> 8.32 mm
- net /PC6: track 6.10 -> 0.00 mm
- net /PA8: track 6.10 -> 0.00 mm
Changed lines of the file:
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@@
   (general
     (links 7)
-    (no_connects 1)
+    (no_connects 3)
     (area 96.266 79.121 266.827001 205.740001)
     (thickness 1.6)
@@
   )
   (net 0 "")
-  (net 1 /PA8)
-  (net 2 /PC6)
+  (net 1 /CAM)
+  (net 2 /CRANK)
   (net 3 CAN_RX)
   (net 4 GND)
@@
     (uvia_drill 0.127)
     (add_net "")
-    (add_net /PA8)
-    (add_net /PC6)
+    (add_net /CAM)
+    (add_net /CRANK)
     (add_net CAN_RX)
     (add_net GND)
@@
     (descr "Double rangee de contacts 2 x 4 pins")
     (tags CONN)
-    (fp_text reference P1 (at 0 -3.81 270) (layer F.SilkS)
+    (fp_text reference P51 (at 0 -3.81 270) (layer F.SilkS)
       (effects (font (size 1.016 1.016) (thickness 0.2032)))
     )
@@
     (pad 1 thru_hole rect (at -3.81 1.27 270) (size 1.524 1.524) (drill 1.016)
       (layers *.Cu *.Mask F.SilkS)
-      (net 1 /PA8)
+      (net 2 /CRANK)
     )
     (pad 2 thru_hole circle (at -3.81 -1.27 270) (size 1.524 1.524) (drill 1.016)
@@
     (pad 5 thru_hole circle (at 1.27 1.27 270) (size 1.524 1.524) (drill 1.016)
       (layers *.Cu *.Mask F.SilkS)
-      (net 2 /PC6)
+      (net 1 /CAM)
     )
     (pad 6 thru_hole circle (at 1.27 -1.27 270) (size 1.524 1.524) (drill 1.016)
@@
     (descr "Double rangee de contacts 2 x 5 pins")
     (tags CONN)
-    (fp_text reference P4 (at 0.635 -3.81 90) (layer F.SilkS)
+    (fp_text reference P54 (at 0.635 -3.81 90) (layer F.SilkS)
       (effects (font (size 1.016 1.016) (thickness 0.2032)))
     )
@@
     (descr "Connecteurs 2 pins")
     (tags "CONN DEV")
-    (fp_text reference P3 (at 0 -1.905) (layer F.SilkS)
+    (fp_text reference P53 (at 0 -1.905) (layer F.SilkS)
       (effects (font (size 0.762 0.762) (thickness 0.1524)))
     )
@@
     )
   )
-  (module SIL-2 (layer F.Cu)
-    (at 170.434 185.42)
-    (descr "Connecteurs 2 pins")
-    (tags "CONN DEV")
-    (fp_text reference W1 (at 0 -2.54) (layer F.SilkS)
-      (effects (font (size 1.72974 1.08712) (thickness 0.3048)))
-    )
-    (fp_text value TEST (at 0 -2.54) (layer F.SilkS) hide
-      (effects (font (size 1.524 1.016) (thickness 0.3048)))
-    )
-    (fp_line (start -2.54 1.27) (end -2.54 -1.27) (layer F.SilkS) (width 0.3048))
-    (fp_line (start -2.54 -1.27) (end 2.54 -1.27) (layer F.SilkS) (width 0.3048))
-    (fp_line (start 2.54 -1.27) (end 2.54 1.27) (layer F.SilkS) (width 0.3048))
-    (fp_line (start 2.54 1.27) (end -2.54 1.27) (layer F.SilkS) (width 0.3048))
-    (pad 1 thru_hole rect (at -1.27 0) (size 1.397 1.397) (drill 0.8128)
-      (layers *.Cu *.Mask F.SilkS)
-    )
-    (pad 2 thru_hole circle (at 1.27 0) (size 1.397 1.397) (drill 0.8128)
-      (layers *.Cu *.Mask F.SilkS)
-      (net 2 /PC6)
-    )
-  )
-  (module SIL-2 (layer F.Cu)
-    (at 170.434 180.34)
-    (descr "Connecteurs 2 pins")
-    (tags "CONN DEV")
-    (fp_text reference W2 (at 0 -2.54) (layer F.SilkS)
-      (effects (font (size 1.72974 1.08712) (thickness 0.3048)))
-    )
-    (fp_text value TEST (at 0 -2.54) (layer F.SilkS) hide
-      (effects (font (size 1.524 1.016) (thickness 0.3048)))
-    )
-    (fp_line (start -2.54 1.27) (end -2.54 -1.27) (layer F.SilkS) (width 0.3048))
-    (fp_line (start -2.54 -1.27) (end 2.54 -1.27) (layer F.SilkS) (width 0.3048))
-    (fp_line (start 2.54 -1.27) (end 2.54 1.27) (layer F.SilkS) (width 0.3048))
-    (fp_line (start 2.54 1.27) (end -2.54 1.27) (layer F.SilkS) (width 0.3048))
-    (pad 1 thru_hole rect (at -1.27 0) (size 1.397 1.397) (drill 0.8128)
-      (layers *.Cu *.Mask F.SilkS)
-    )
-    (pad 2 thru_hole circle (at 1.27 0) (size 1.397 1.397) (drill 0.8128)
-      (layers *.Cu *.Mask F.SilkS)
-      (net 1 /PA8)
-    )
-  )
-  (module SIL-2 (layer F.Cu)
-    (at 135.509 170.18)
-    (descr "Connecteurs 2 pins")
-    (tags "CONN DEV")
-    (fp_text reference W3 (at 0 -2.54) (layer F.SilkS)
-      (effects (font (size 1.72974 1.08712) (thickness 0.3048)))
-    )
-    (fp_text value TEST (at 0 -2.54) (layer F.SilkS) hide
-      (effects (font (size 1.524 1.016) (thickness 0.3048)))
-    )
-    (fp_line (start -2.54 1.27) (end -2.54 -1.27) (layer F.SilkS) (width 0.3048))
-    (fp_line (start -2.54 -1.27) (end 2.54 -1.27) (layer F.SilkS) (width 0.3048))
-    (fp_line (start 2.54 -1.27) (end 2.54 1.27) (layer F.SilkS) (width 0.3048))
-    (fp_line (start 2.54 1.27) (end -2.54 1.27) (layer F.SilkS) (width 0.3048))
-    (pad 1 thru_hole rect (at -1.27 0) (size 1.397 1.397) (drill 0.8128)
-      (layers *.Cu *.Mask F.SilkS)
-      (net 3 CAN_RX)
-    )
-    (pad 2 thru_hole circle (at 1.27 0) (size 1.397 1.397) (drill 0.8128)
-      (layers *.Cu *.Mask F.SilkS)
-      (net 3 CAN_RX)
-    )
-  )
   (module PIN_ARRAY_10X2_M (layer F.Cu)
     (at 128.27 176.53 270)
-    (fp_text reference P2 (at 0 -3.81 270) (layer F.SilkS)
+    (fp_text reference P52 (at 0 -3.81 270) (layer F.SilkS)
       (effects (font (size 1.016 1.016) (thickness 0.254)))
     )
@@
       (scale (xyz 1 1 1))
       (rotate (xyz -90 0 0))
+    )
+  )
+  (module SIL-2 (layer F.Cu)
+    (at 173.482 180.34 180)
+    (descr "Connecteurs 2 pins")
+    (tags "CONN DEV")
+    (fp_text reference JP1 (at 0 -2.54 180) (layer F.SilkS)
+      (effects (font (size 1.72974 1.08712) (thickness 0.3048)))
+    )
+    (fp_text value JUMPER (at 0 -2.54 180) (layer F.SilkS) hide
+      (effects (font (size 1.524 1.016) (thickness 0.3048)))
+    )
+    (fp_line (start -2.54 1.27) (end -2.54 -1.27) (layer F.SilkS) (width 0.3048))
+    (fp_line (start -2.54 -1.27) (end 2.54 -1.27) (layer F.SilkS) (width 0.3048))
+    (fp_line (start 2.54 -1.27) (end 2.54 1.27) (layer F.SilkS) (width 0.3048))
+    (fp_line (start 2.54 1.27) (end -2.54 1.27) (layer F.SilkS) (width 0.3048))
+    (pad 1 thru_hole rect (at -1.27 0 180) (size 1.397 1.397) (drill 0.8128)
+      (layers *.Cu *.Mask F.SilkS)
+    )
+    (pad 2 thru_hole circle (at 1.27 0 180) (size 1.397 1.397) (drill 0.8128)
+      (layers *.Cu *.Mask F.SilkS)
+      (net 2 /CRANK)
+    )
+  )
+  (module SIL-2 (layer F.Cu)
+    (at 171.196 185.42 180)
+    (descr "Connecteurs 2 pins")
+    (tags "CONN DEV")
+    (fp_text reference JP2 (at 0 -2.54 180) (layer F.SilkS)
+      (effects (font (size 1.72974 1.08712) (thickness 0.3048)))
+    )
+    (fp_text value JUMPER (at 0 -2.54 180) (layer F.SilkS) hide
+      (effects (font (size 1.524 1.016) (thickness 0.3048)))
+    )
+    (fp_line (start -2.54 1.27) (end -2.54 -1.27) (layer F.SilkS) (width 0.3048))
+    (fp_line (start -2.54 -1.27) (end 2.54 -1.27) (layer F.SilkS) (width 0.3048))
+    (fp_line (start 2.54 -1.27) (end 2.54 1.27) (layer F.SilkS) (width 0.3048))
+    (fp_line (start 2.54 1.27) (end -2.54 1.27) (layer F.SilkS) (width 0.3048))
+    (pad 1 thru_hole rect (at -1.27 0 180) (size 1.397 1.397) (drill 0.8128)
+      (layers *.Cu *.Mask F.SilkS)
+    )
+    (pad 2 thru_hole circle (at 1.27 0 180) (size 1.397 1.397) (drill 0.8128)
+      (layers *.Cu *.Mask F.SilkS)
+      (net 1 /CAM)
+    )
+  )
+  (module SIL-2 (layer F.Cu)
+    (at 135.5725 170.2435 180)
+    (descr "Connecteurs 2 pins")
+    (tags "CONN DEV")
+    (fp_text reference JP3 (at 0 -2.54 180) (layer F.SilkS)
+      (effects (font (size 1.72974 1.08712) (thickness 0.3048)))
+    )
+    (fp_text value JUMPER (at 0 -2.54 180) (layer F.SilkS) hide
+      (effects (font (size 1.524 1.016) (thickness 0.3048)))
+    )
+    (fp_line (start -2.54 1.27) (end -2.54 -1.27) (layer F.SilkS) (width 0.3048))
+    (fp_line (start -2.54 -1.27) (end 2.54 -1.27) (layer F.SilkS) (width 0.3048))
+    (fp_line (start 2.54 -1.27) (end 2.54 1.27) (layer F.SilkS) (width 0.3048))
+    (fp_line (start 2.54 1.27) (end -2.54 1.27) (layer F.SilkS) (width 0.3048))
+    (pad 1 thru_hole rect (at -1.27 0 180) (size 1.397 1.397) (drill 0.8128)
+      (layers *.Cu *.Mask F.SilkS)
+      (net 3 CAN_RX)
+    )
+    (pad 2 thru_hole circle (at 1.27 0 180) (size 1.397 1.397) (drill 0.8128)
+      (layers *.Cu *.Mask F.SilkS)
+      (net 3 CAN_RX)
     )
   )
@@
   (gr_line (start 127 187.96) (end 129.54 187.96) (angle 90) (layer Cmts.User) (width 0.2))
   (gr_line (start 127 127) (end 127 187.96) (angle 90) (layer Cmts.User) (width 0.2))
-  (segment (start 171.704 180.34) (end 177.8 180.34) (width 0.254) (layer F.Cu) (net 1))
-  (segment (start 171.704 185.42) (end 177.8 185.42) (width 0.254) (layer F.Cu) (net 2))
+  (segment (start 172.466 185.42) (end 177.8 185.42) (width 0.254) (layer F.Cu) (net 0) (status 10))
+  (segment (start 174.8155 180.34) (end 177.8 180.34) (width 0.254) (layer F.Cu) (net 0) (status 10))
   (segment (start 134.239 170.18) (end 129.54 170.18) (width 0.254) (layer F.Cu) (net 3))
   (zone (net 4) (net_name GND) (layer F.Cu) (hatch edge 0.508)

Commit message: making progress
Parts:
- added P55: CONN_2, PIN_ARRAY_2X1, F.Cu at (203.5, 182.8)
- added P56: CONN_6, PIN_ARRAY-6X1, F.Cu at (121.9, 181.5)
- added P57: CONN_6, PIN_ARRAY-6X1, F.Cu at (121.9, 166.4)
- moved JP2 2.41 mm to (173.6, 185.4)
- moved JP3 1.91 mm to (133.7, 170.1)
- moved JP1 0.13 mm to (173.6, 180.3)
Connections:
- P51 pad 4: (no net) -> /PC9
- P51 pad 6: (no net) -> /PC7
- P52 pad 1: (no net) -> /PE13
- P52 pad 10: (no net) -> /PD8
- P52 pad 11: (no net) -> /PD9
- P52 pad 12: (no net) -> /PD10
- P52 pad 13: (no net) -> /PD11
- P52 pad 3: (no net) -> /PE15
- P52 pad 4: (no net) -> /PB10
- P52 pad 5: (no net) -> /PB11
- P52 pad 7: (no net) -> /PB13
- P52 pad 8: (no net) -> /PB14
- P52 pad 9: (no net) -> /PB15
Routing:
- net /PD11: track 0.00 -> 5.12 mm
- net /PB15: track 0.00 -> 5.12 mm
- net /PD9: track 0.00 -> 5.10 mm
- net /PE15: track 0.00 -> 5.10 mm
- net /PE13: track 0.00 -> 5.10 mm
- net /PB13: track 0.00 -> 5.10 mm
- net /PB11: track 0.00 -> 5.10 mm
- net (no net): track 8.32 -> 5.78 mm
- net CAN_RX: track 4.70 -> 2.80 mm
Other:
- board text added: "BOOT0"
- board text added: "CAN RX"
- board text added: "GND"
- board text added: "PB11"
- board text added: "PB13"
- board text added: "PB15"
- board text added: "PD11"
- board text added: "PD9"
- board text added: "PE13"
- board text added: "PE15"
- board text added: "VDD"

Commit message: making progress
Parts:
- added P58: CONN_6, PIN_ARRAY-6X1, F.Cu at (139.8, 190.1)
- moved JP3 0.14 mm to (133.5, 170.2)
- moved JP1 0.06 mm to (173.5, 180.3), turned to 0 degrees
- turned JP2 to 0 degrees
- turned P54 to 270 degrees
Connections:
- net /CAM renamed /PC6
- net /CRANK renamed /PA8
- JP3 pad 1: CAN_RX -> (no net)
- JP3 pad 2: CAN_RX -> /PB12
- P52 pad 6: CAN_RX -> /PB12
- P54 pad 7: (no net) -> /PE9
- P54 pad 9: (no net) -> /PE11
- P57 pad 5: /PB14 -> /PE11
- P57 pad 6: /PB10 -> /PE9
Routing:
- net /PD8: track 0.00 -> 14.6 mm
- net /PD10: track 0.00 -> 12.7 mm
- net (no net): track 5.78 -> 0.00 mm
- net /PE9: track 0.00 -> 5.08 mm
- net /PE11: track 0.00 -> 5.08 mm
- net /PC6: track 0.00 -> 2.92 mm
- net /PA8: track 0.00 -> 2.86 mm
- net CAN_RX: track 2.80 -> 0.00 mm
- net /PB12: track 0.00 -> 2.67 mm
Other:
- board text added: "PB10"
- board text added: "PB12"
- board text added: "PB14"
- board text added: "PD10"
- board text added: "PD8"
- board text added: "PE11"
- board text added: "PE9"

Commit message: making progress
Parts:
- removed JP1, JP2, JP3: JUMPER, SIL-2
- added JP51: JUMPER, PIN_ARRAY_2_A, F.Cu at (134.0, 170.2)
- added JP52: JUMPER, PIN_ARRAY_2_A, F.Cu at (173.3, 180.3)
- added JP53: JUMPER, PIN_ARRAY_2_A, F.Cu at (173.2, 185.4)
- added P_VOID1: CONN_6, PIN_ARRAY-6X1, F.Cu at (156.5, 217.2)
