File: trunk/hardware/frankenstein_foundation/frankenstein_foundation.kicad_pcb (KiCad board)
At the start: 2 copper layers, 100 x 99.9 mm, 12 parts, among them P51 CONN_4X2, P52 CONN_10X2, P53 CONN_2, P54 CONN_5X2, P55 CONN_2, P56 CONN_6, P57 CONN_6, P58 CONN_6

Commit message: making progress
Parts:
- P55: value CONN_2 -> CONN_6; footprint PIN_ARRAY_2X1 -> PIN_ARRAY-6X1
- moved P55 30.5 mm to (174.0, 190.6), turned to 180 degrees
Connections:
- P55 pad 1: /PC7 -> (no net)
Changed lines of the file:
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@@
 (kicad_pcb (version 3) (host pcbnew "(2013-07-07 BZR 4022)-stable")
   (general
-    (links 25)
+    (links 27)
     (no_connects 7)
     (area 96.266 79.121 266.827001 220.1418)
     (thickness 1.6)
     (drawings 56)
-    (tracks 32)
+    (tracks 33)
     (zones 0)
     (modules 12)
@@
     )
   )
-  (module PIN_ARRAY_2X1 (layer F.Cu)
-    (at 203.5175 182.753)
-    (descr "Connecteurs 2 pins")
-    (tags "CONN DEV")
-    (fp_text reference P55 (at 0 -1.905) (layer F.SilkS)
-      (effects (font (size 0.762 0.762) (thickness 0.1524)))
-    )
-    (fp_text value CONN_2 (at 0 -1.905) (layer F.SilkS) hide
-      (effects (font (size 0.762 0.762) (thickness 0.1524)))
-    )
-    (fp_line (start -2.54 1.27) (end -2.54 -1.27) (layer F.SilkS) (width 0.1524))
-    (fp_line (start -2.54 -1.27) (end 2.54 -1.27) (layer F.SilkS) (width 0.1524))
-    (fp_line (start 2.54 -1.27) (end 2.54 1.27) (layer F.SilkS) (width 0.1524))
-    (fp_line (start 2.54 1.27) (end -2.54 1.27) (layer F.SilkS) (width 0.1524))
-    (pad 1 thru_hole rect (at -1.27 0) (size 1.524 1.524) (drill 1.016)
-      (layers *.Cu *.Mask F.SilkS)
-      (net 12 /PC7)
-    )
-    (pad 2 thru_hole circle (at 1.27 0) (size 1.524 1.524) (drill 1.016)
-      (layers *.Cu *.Mask F.SilkS)
-      (net 13 /PC9)
-    )
-    (model pin_array/pins_array_2x1.wrl
-      (at (xyz 0 0 0))
-      (scale (xyz 1 1 1))
-      (rotate (xyz 0 0 0))
-    )
-  )
   (module PIN_ARRAY-6X1 (layer F.Cu)
     (at 121.92 181.483 90)
@@
     )
   )
+  (module PIN_ARRAY-6X1 (layer F.Cu)
+    (at 173.99 190.5635 180)
+    (descr "Connecteur 6 pins")
+    (tags "CONN DEV")
+    (fp_text reference P55 (at 0 -2.159 180) (layer F.SilkS)
+      (effects (font (size 1.016 1.016) (thickness 0.2032)))
+    )
+    (fp_text value CONN_6 (at 0 2.159 180) (layer F.SilkS) hide
+      (effects (font (size 1.016 0.889) (thickness 0.2032)))
+    )
+    (fp_line (start -7.62 1.27) (end -7.62 -1.27) (layer F.SilkS) (width 0.3048))
+    (fp_line (start -7.62 -1.27) (end 7.62 -1.27) (layer F.SilkS) (width 0.3048))
+    (fp_line (start 7.62 -1.27) (end 7.62 1.27) (layer F.SilkS) (width 0.3048))
+    (fp_line (start 7.62 1.27) (end -7.62 1.27) (layer F.SilkS) (width 0.3048))
+    (fp_line (start -5.08 1.27) (end -5.08 -1.27) (layer F.SilkS) (width 0.3048))
+    (pad 1 thru_hole rect (at -6.35 0 180) (size 1.524 1.524) (drill 1.016)
+      (layers *.Cu *.Mask F.SilkS)
+    )
+    (pad 2 thru_hole circle (at -3.81 0 180) (size 1.524 1.524) (drill 1.016)
+      (layers *.Cu *.Mask F.SilkS)
+      (net 13 /PC9)
+    )
+    (pad 3 thru_hole circle (at -1.27 0.0635 180) (size 1.524 1.524) (drill 1.016)
+      (layers *.Cu *.Mask F.SilkS)
+      (net 12 /PC7)
+    )
+    (pad 4 thru_hole circle (at 1.27 0 180) (size 1.524 1.524) (drill 1.016)
+      (layers *.Cu *.Mask F.SilkS)
+      (net 22 GND)
+    )
+    (pad 5 thru_hole circle (at 3.81 0 180) (size 1.524 1.524) (drill 1.016)
+      (layers *.Cu *.Mask F.SilkS)
+      (net 22 GND)
+    )
+    (pad 6 thru_hole circle (at 6.35 0 180) (size 1.524 1.524) (drill 1.016)
+      (layers *.Cu *.Mask F.SilkS)
+    )
+    (model pin_array/pins_array_6x1.wrl
+      (at (xyz 0 0 0))
+      (scale (xyz 1 1 1))
+      (rotate (xyz 0 0 0))
+    )
+  )
   (gr_text PB13 (at 124.5235 172.2755) (layer B.SilkS)
     (effects (font (size 0.508 0.508) (thickness 0.127)) (justify mirror))
@@
     (effects (font (size 0.508 0.508) (thickness 0.127)))
   )
-  (gr_text GND (at 180.2765 189.992) (layer F.SilkS)
-    (effects (font (size 0.508 0.508) (thickness 0.127)))
-  )
-  (gr_text GND (at 177.673 189.9285) (layer F.SilkS)
+  (gr_text GND (at 180.975 191.389) (layer F.SilkS)
+    (effects (font (size 0.508 0.508) (thickness 0.127)))
+  )
+  (gr_text GND (at 177.165 189.8015) (layer F.SilkS)
     (effects (font (size 0.508 0.508) (thickness 0.127)))
   )
@@
   (segment (start 122.00636 175.21936) (end 121.92 175.133) (width 0.254) (layer F.Cu) (net 10))
   (segment (start 174.752 185.293) (end 177.8 185.42) (width 0.254) (layer F.Cu) (net 11) (status 10))
+  (segment (start 180.34 185.42) (end 180.5305 185.42) (width 0.254) (layer F.Cu) (net 12))
   (segment (start 129.54 177.75936) (end 129.45364 177.75936) (width 0.254) (layer B.Cu) (net 14))
   (segment (start 124.1425 183.0705) (end 121.92 185.293) (width 0.254) (layer B.Cu) (net 14))
