File: hardware/1A_injector_12-channels/inj_12ch.kicad_pcb (KiCad board)
At the start: 2 copper layers, 47 x 58.9 mm, 58 parts, among them P1 CONN_3, P2 CONN_10X2, P3 CONN_16, P4 CONN_1, P5 CONN_1, Q1 OVP_DRIVER, Q10 OVP_DRIVER, Q11 OVP_DRIVER, Q12 OVP_DRIVER, Q2 OVP_DRIVER, Q3 OVP_DRIVER, Q4 OVP_DRIVER, Q5 OVP_DRIVER, Q6 OVP_DRIVER, Q7 OVP_DRIVER, Q8 OVP_DRIVER, Q9 OVP_DRIVER

Commit message: a version for F
Parts:
- added M401: CONN_1, 1pin, F.Cu at (210.8, 95.2)
- renumbered D1 to D401, D2 to D402, D3 to D403, D4 to D404, D5 to D405, D6 to D406, D7 to D407, D8 to D408, D9 to D409, D10 to D410, D11 to D411, D12 to D412, D13 to D413, D14 to D414, P1 to P401, P2 to P402, P3 to P403, P4 to P404, P5 to P405, Q1 to Q401, Q2 to Q402, Q3 to Q403, Q4 to Q404, Q5 to Q405, Q6 to Q406, Q7 to Q407, Q8 to Q408, Q9 to Q409, Q10 to Q410, Q11 to Q411, Q12 to Q412, R1 to R401, R2 to R402, R3 to R403, R4 to R404, R5 to R405, R6 to R406, R7 to R407, R8 to R408, R9 to R409, R10 to R410, R11 to R411, R12 to R412, R13 to R413, R14 to R414, R15 to R415, R16 to R416, R17 to R417, R18 to R418, R19 to R419, R20 to R420, R21 to R421, R22 to R422, R23 to R423, R24 to R424, R25 to R425, R26 to R426, R27 to R427
Connections:
- P401 pad 2: /5V -> /3.3V
- P401 pad 3: /3.3V -> /5V
Routing:
- net GND: track 468.2 -> 465.5 mm, vias 196 -> 195
- net /5V: track 65.2 -> 62.6 mm, vias 0 -> 1
- net /3.3V: track 49.9 -> 49.2 mm
Other:
- outline, holes or cut-outs redrawn
- net class .02 added: clearance 0.2032, trace_width 0.508, via_dia 0.889, via_drill 0.635
- net class 10A EXT removed
- net class 10A INT removed
- net class 10A INT MOD removed
- net class 1A EXT removed
- net class 1A INT removed
- net class 5A EXT removed
- net class 5A INT removed
- net class Default: clearance 0.254 -> 0.2032; via_dia 1.016 -> 0.889; via_drill 0.508 -> 0.635
- rule pad_to_mask_clearance: 0.254 -> 0
- rule trace_clearance: 0.254 -> 0.2032
- rule trace_min: 0.1524 -> 0.254
- rule via_min_size: 1.016 -> 0.889
- board text added: "5V 3V GND"
- board text added: "BAT"
