File: hardware/284617-1-connector/284617-1.kicad_pcb (KiCad board)
At the start: 2 copper layers, 150 x 50 mm, 1 part, among them P1 284617-1

Commit message: initial version
Parts:
- added P10: CONN_5, PIN_ARRAY_5x1, F.Cu at (99.1, 108.0)
- added P11: CONN_9, PIN_ARRAY_9x1, F.Cu at (124.5, 108.0)
- added P12: CONN_5, PIN_ARRAY_5x1, F.Cu at (99.1, 111.8)
- added P13: CONN_9, PIN_ARRAY_9x1, F.Cu at (124.5, 111.8)
- added P14: CONN_22, PIN_ARRAY_22x1, F.Cu at (188.0, 101.6)
- added P15: CONN_22, PIN_ARRAY_22x1, F.Cu at (188.0, 105.4)
- added P16: CONN_22, PIN_ARRAY_22x1, F.Cu at (188.0, 109.2)
- added P17: CONN_22, PIN_ARRAY_22x1, F.Cu at (188.0, 113.0)
- added P18: CONN_1, 1pin(m), F.Cu at (144.8, 99.1)
- added P19: CONN_1, 1pin(m), F.Cu at (152.4, 99.1)
- added P2: CONN_1, PIN_ARRAY_1, F.Cu at (135.9, 100.3)
- added P20: CONN_1, 1pin(m), F.Cu at (144.8, 105.4)
- added P21: CONN_1, 1pin(m), F.Cu at (152.4, 105.4)
- added P22: CONN_1, 1pin(m), F.Cu at (144.8, 111.8)
- added P23: CONN_1, 1pin(m), F.Cu at (152.4, 111.8)
- added P24: CONN_1, 1pin, F.Cu at (222.0, 98.0)
- added P25: CONN_1, 1pin, F.Cu at (78.0, 98.0)
- added P3: CONN_1, PIN_ARRAY_1, F.Cu at (135.9, 104.1)
- added P4: CONN_1, PIN_ARRAY_1, F.Cu at (135.9, 108.0)
- added P5: CONN_1, PIN_ARRAY_1, F.Cu at (135.9, 111.8)
- added P6: CONN_5, PIN_ARRAY_5x1, F.Cu at (99.1, 100.3)
- added P7: CONN_9, PIN_ARRAY_9x1, F.Cu at (124.5, 100.3)
- added P8: CONN_5, PIN_ARRAY_5x1, F.Cu at (99.1, 104.1)
- added P9: CONN_9, PIN_ARRAY_9x1, F.Cu at (124.5, 104.1)
- moved P1 0.75 mm to (72.5, 115.8)
Connections:
- P1 pad 1: (no net) -> N-0000097
- P1 pad 10: (no net) -> N-00000120
- P1 pad 100: (no net) -> N-0000010
- P1 pad 101: (no net) -> N-000009
- P1 pad 102: (no net) -> N-000008
- P1 pad 103: (no net) -> N-000007
- P1 pad 104: (no net) -> N-000006
- P1 pad 105: (no net) -> N-000005
- P1 pad 106: (no net) -> N-000004
- P1 pad 107: (no net) -> N-000003
- P1 pad 108: (no net) -> N-000002
- P1 pad 109: (no net) -> N-0000016
- P1 pad 11: (no net) -> N-00000114
- P1 pad 110: (no net) -> N-0000059
- P1 pad 111: (no net) -> N-0000058
- P1 pad 112: (no net) -> N-0000057
- P1 pad 113: (no net) -> N-0000056
- P1 pad 114: (no net) -> N-0000055
- P1 pad 115: (no net) -> N-0000054
- P1 pad 116: (no net) -> N-0000053
- P1 pad 117: (no net) -> N-0000052
- P1 pad 118: (no net) -> N-0000051
- P1 pad 119: (no net) -> N-0000050
- P1 pad 12: (no net) -> N-00000109
- P1 pad 120: (no net) -> N-0000049
- P1 pad 121: (no net) -> N-0000048
- P1 pad 122: (no net) -> N-0000047
- P1 pad 123: (no net) -> N-0000031
- P1 pad 124: (no net) -> N-0000045
- P1 pad 125: (no net) -> N-0000044
- P1 pad 126: (no net) -> N-0000043
- P1 pad 127: (no net) -> N-0000042
- P1 pad 128: (no net) -> N-0000041
- P1 pad 129: (no net) -> N-0000040
- P1 pad 13: (no net) -> N-00000104
- P1 pad 130: (no net) -> N-0000039
- P1 pad 131: (no net) -> N-0000038
- P1 pad 132: (no net) -> N-0000037
- P1 pad 133: (no net) -> N-0000036
- P1 pad 134: (no net) -> N-0000035
- P1 pad 135: (no net) -> N-0000034
- P1 pad 136: (no net) -> N-0000033
- P1 pad 137: (no net) -> N-0000032
- P1 pad 138: (no net) -> N-0000060
- P1 pad 139: (no net) -> N-0000086
- P1 pad 14: (no net) -> N-00000155
- P1 pad 140: (no net) -> N-0000082
- P1 pad 141: (no net) -> N-0000080
- P1 pad 142: (no net) -> N-0000078
- P1 pad 143: (no net) -> N-0000076
- P1 pad 144: (no net) -> N-0000074
- P1 pad 145: (no net) -> N-0000089
- P1 pad 146: (no net) -> N-0000088
- P1 pad 147: (no net) -> N-0000083
- P1 pad 148: (no net) -> N-0000087
- P1 pad 149: (no net) -> N-0000085
- P1 pad 15: (no net) -> N-00000150
- P1 pad 150: (no net) -> N-0000081
- P1 pad 151: (no net) -> N-0000079
- P1 pad 152: (no net) -> N-0000077
- P1 pad 153: (no net) -> N-0000075
- P1 pad 154: (no net) -> N-0000073
- P1 pad 16: (no net) -> N-00000146
- P1 pad 17: (no net) -> N-00000141
- P1 pad 18: (no net) -> N-00000136
- P1 pad 19: (no net) -> N-00000132
- P1 pad 2: (no net) -> N-00000128
- P1 pad 20: (no net) -> N-00000119
- P1 pad 21: (no net) -> N-00000113
- P1 pad 22: (no net) -> N-00000108
- P1 pad 23: (no net) -> N-00000103
- P1 pad 24: (no net) -> N-00000154
- P1 pad 25: (no net) -> N-00000149
- P1 pad 26: (no net) -> N-00000145
- P1 pad 27: (no net) -> N-00000140
- P1 pad 28: (no net) -> N-00000135
- P1 pad 29: (no net) -> N-00000131
- P1 pad 3: (no net) -> N-00000127
- P1 pad 30: (no net) -> N-00000118
- P1 pad 31: (no net) -> N-00000112
- P1 pad 32: (no net) -> N-00000107
- P1 pad 33: (no net) -> N-00000102
- P1 pad 34: (no net) -> N-00000153
- P1 pad 35: (no net) -> N-00000148
- P1 pad 36: (no net) -> N-00000144
- P1 pad 37: (no net) -> N-00000139
- P1 pad 38: (no net) -> N-00000134
- P1 pad 39: (no net) -> N-00000130
- P1 pad 4: (no net) -> N-00000126
- P1 pad 40: (no net) -> N-00000117
- P1 pad 41: (no net) -> N-00000111
- P1 pad 42: (no net) -> N-00000106
- P1 pad 43: (no net) -> N-00000101
- P1 pad 44: (no net) -> N-00000152
- P1 pad 45: (no net) -> N-0000092
- P1 pad 46: (no net) -> N-00000129
- P1 pad 47: (no net) -> N-00000138
- P1 pad 48: (no net) -> N-00000133
- P1 pad 49: (no net) -> N-0000099
- P1 pad 5: (no net) -> N-00000125
- P1 pad 50: (no net) -> N-00000116
- P1 pad 51: (no net) -> N-00000110
- P1 pad 52: (no net) -> N-00000105
- P1 pad 53: (no net) -> N-00000115
- P1 pad 54: (no net) -> N-00000151
- P1 pad 55: (no net) -> N-00000147
- P1 pad 56: (no net) -> N-00000142
- P1 pad 57: (no net) -> N-00000137
- P1 pad 58: (no net) -> N-00000143
- P1 pad 59: (no net) -> N-0000098
- P1 pad 6: (no net) -> N-00000124
- P1 pad 60: (no net) -> N-00000100
- P1 pad 61: (no net) -> N-0000091
- P1 pad 62: (no net) -> N-0000090
- P1 pad 63: (no net) -> N-0000093
- P1 pad 64: (no net) -> N-0000096
- P1 pad 65: (no net) -> N-0000095
- P1 pad 66: (no net) -> N-0000094
- P1 pad 67: (no net) -> N-0000072
- P1 pad 68: (no net) -> N-0000071
- P1 pad 69: (no net) -> N-0000070
- P1 pad 7: (no net) -> N-00000123
- P1 pad 70: (no net) -> N-0000069
- P1 pad 71: (no net) -> N-0000068
- P1 pad 72: (no net) -> N-0000067
- P1 pad 73: (no net) -> N-0000066
- P1 pad 74: (no net) -> N-0000065
- P1 pad 75: (no net) -> N-0000064
- P1 pad 76: (no net) -> N-0000063
- P1 pad 77: (no net) -> N-0000062
- P1 pad 78: (no net) -> N-0000061
- P1 pad 79: (no net) -> N-0000046
- P1 pad 8: (no net) -> N-00000122
- P1 pad 80: (no net) -> N-0000030
- P1 pad 81: (no net) -> N-0000029
- P1 pad 82: (no net) -> N-0000028
- P1 pad 83: (no net) -> N-0000027
- P1 pad 84: (no net) -> N-0000026
- P1 pad 85: (no net) -> N-0000025
- P1 pad 86: (no net) -> N-0000024
- P1 pad 87: (no net) -> N-0000023
- P1 pad 88: (no net) -> N-0000022
- P1 pad 89: (no net) -> N-0000021
- P1 pad 9: (no net) -> N-00000121
- P1 pad 90: (no net) -> N-0000020
- P1 pad 91: (no net) -> N-0000019
- P1 pad 92: (no net) -> N-0000018
- P1 pad 93: (no net) -> N-0000017
- P1 pad 94: (no net) -> N-000001
- P1 pad 95: (no net) -> N-0000015
- P1 pad 96: (no net) -> N-0000014
- P1 pad 97: (no net) -> N-0000013
- P1 pad 98: (no net) -> N-0000012
- P1 pad 99: (no net) -> N-0000011
Routing:
- net N-0000064: track 0.00 -> 126.8 mm
- net N-0000063: track 0.00 -> 122.7 mm
- net N-00000114: track 0.00 -> 122.3 mm
- net N-00000120: track 0.00 -> 117.2 mm
- net N-0000062: track 0.00 -> 113.8 mm
- net N-00000121: track 0.00 -> 109.1 mm
- net N-0000061: track 0.00 -> 108.7 mm
- net N-00000122: track 0.00 -> 106.4 mm
- net N-0000046: track 0.00 -> 100.6 mm
- net N-0000030: track 0.00 -> 95.5 mm
- net N-0000029: track 0.00 -> 87.4 mm
- net N-0000065: track 0.00 -> 86.5 mm
- net N-0000028: track 0.00 -> 82.3 mm
- net N-0000066: track 0.00 -> 81.8 mm
- net N-00000125: track 0.00 -> 78.3 mm
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- added copper zone on B.Cu, net /GND
- added copper zone on F.Cu, net /GND
Other:
- net class 1.5A added: clearance 0.254, trace_width 0.49, via_dia 0.889, via_drill 0.635
- net class 1A added: clearance 0.254, trace_width 0.3, via_dia 0.889, via_drill 0.635
- net class 4A added: clearance 0.254, trace_width 2, via_dia 0.889, via_drill 0.635
- net class Default: trace_width 0.254 -> 0.3
- board text added: "1"
- board text added: "16"
- board text added: "2"
- board text added: "29"
- board text added: "3"
- board text added: "31"
- board text added: "4"
- board text added: "46"
- board text added: "5"
- board text added: "51"
- board text added: "6"
- board text added: "7"
- board text added: "73"
