File: hardware/frankenso_foundation/frankenso_foundation.kicad_pcb (KiCad board)
At the start: 2 copper layers, 1 part, among them P99 0176122-06

Commit message: making progress
Parts:
- added P_VOID3: CONN_8, pin_array_8x2, F.Cu at (275.6, 171.7)
- added W1: TEST, SM0805_jumper, F.Cu at (214.7, 122.9)
- added W2: TEST, SM0805_jumper, F.Cu at (208.6, 129.5)
- added W3: TEST, SM0805_jumper, F.Cu at (200.7, 125.6)
Connections:
- P99 pad 1: (no net) -> N-000003
- P99 pad 2: (no net) -> N-000004
- P99 pad 3: (no net) -> N-000002
Changed lines of the file:
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@@
 (kicad_pcb (version 3) (host pcbnew "(2013-07-07 BZR 4022)-stable")
   (general
-    (links 0)
-    (no_connects 0)
-    (area 96.266 82.501739 266.827001 265.1695)
+    (links 12)
+    (no_connects 12)
+    (area 0 0 0 0)
     (thickness 1.6)
     (drawings 13)
     (tracks 0)
     (zones 0)
-    (modules 1)
-    (nets 1)
+    (modules 5)
+    (nets 7)
   )
   (page A3)
@@
   )
   (net 0 "")
+  (net 1 /INJ-10)
+  (net 2 /INJ-11)
+  (net 3 /INJ-12)
+  (net 4 N-000002)
+  (net 5 N-000003)
+  (net 6 N-000004)
   (net_class Default "This is the default net class."
     (clearance 0.2032)
@@
     (uvia_drill 0.127)
     (add_net "")
+    (add_net /INJ-10)
+    (add_net /INJ-11)
+    (add_net /INJ-12)
+    (add_net N-000002)
+    (add_net N-000003)
+    (add_net N-000004)
   )
   (module 176122-6 (layer F.Cu)
@@
     (pad 3 thru_hole circle (at -15.25016 0) (size 1.15062 1.15062) (drill 1.09982)
       (layers *.Cu *.Mask F.SilkS)
+      (net 4 N-000002)
     )
     (pad 6 thru_hole circle (at -15.25016 -4.50088 180) (size 1.15062 1.15062) (drill 1.09982)
@@
     (pad 2 thru_hole circle (at -11.75004 0) (size 1.15062 1.15062) (drill 1.09982)
       (layers *.Cu *.Mask F.SilkS)
+      (net 6 N-000004)
     )
     (pad 5 thru_hole circle (at -11.75004 -4.50088 180) (size 1.15062 1.15062) (drill 1.09982)
@@
     (pad 1 thru_hole circle (at -8.24992 0) (size 1.15062 1.15062) (drill 1.09982)
       (layers *.Cu *.Mask F.SilkS)
+      (net 5 N-000003)
     )
     (pad 4 thru_hole circle (at -8.24992 -4.50088 180) (size 1.15062 1.15062) (drill 1.09982)
@@
     )
   )
+  (module SM0805_jumper (layer F.Cu)
+    (at 214.6935 122.8725 270)
+    (attr smd)
+    (fp_text reference W1 (at 0.0635 0 270) (layer F.SilkS)
+      (effects (font (size 0.762 0.762) (thickness 0.127)))
+    )
+    (fp_text value TEST (at 0 1.27 270) (layer F.SilkS) hide
+      (effects (font (size 0.50038 0.50038) (thickness 0.10922)))
+    )
+    (fp_circle (center -1.651 0.762) (end -1.651 0.635) (layer F.SilkS) (width 0.09906))
+    (fp_line (start -0.508 0.762) (end -1.524 0.762) (layer F.SilkS) (width 0.09906))
+    (fp_line (start -1.524 0.762) (end -1.524 -0.762) (layer F.SilkS) (width 0.09906))
+    (fp_line (start -1.524 -0.762) (end -0.508 -0.762) (layer F.SilkS) (width 0.09906))
+    (fp_line (start 0.508 -0.762) (end 1.524 -0.762) (layer F.SilkS) (width 0.09906))
+    (fp_line (start 1.524 -0.762) (end 1.524 0.762) (layer F.SilkS) (width 0.09906))
+    (fp_line (start 1.524 0.762) (end 0.508 0.762) (layer F.SilkS) (width 0.09906))
+    (pad 1 smd rect (at -0.9525 0 270) (size 0.889 1.397)
+      (layers F.Cu F.Paste F.Mask)
+      (net 5 N-000003)
+    )
+    (pad 2 smd rect (at 0.9525 0 270) (size 0.889 1.397)
+      (layers F.Cu F.Paste F.Mask)
+      (net 3 /INJ-12)
+    )
+    (pad 2 thru_hole circle (at 1.905 0 270) (size 1.524 1.524) (drill 0.8128)
+      (layers *.Cu *.Mask F.SilkS)
+      (net 3 /INJ-12)
+    )
+    (pad 1 thru_hole circle (at -1.905 0 270) (size 1.524 1.524) (drill 0.8128)
+      (layers *.Cu *.Mask F.SilkS)
+      (net 5 N-000003)
+    )
+    (model smd/chip_cms.wrl
+      (at (xyz 0 0 0))
+      (scale (xyz 0.1 0.1 0.1))
+      (rotate (xyz 0 0 0))
+    )
+  )
+  (module SM0805_jumper (layer F.Cu)
+    (at 208.5975 129.54 270)
+    (attr smd)
+    (fp_text reference W2 (at 0.0635 0 360) (layer F.SilkS)
+      (effects (font (size 0.762 0.762) (thickness 0.127)))
+    )
+    (fp_text value TEST (at 0 1.27 270) (layer F.SilkS) hide
+      (effects (font (size 0.50038 0.50038) (thickness 0.10922)))
+    )
+    (fp_circle (center -1.651 0.762) (end -1.651 0.635) (layer F.SilkS) (width 0.09906))
+    (fp_line (start -0.508 0.762) (end -1.524 0.762) (layer F.SilkS) (width 0.09906))
+    (fp_line (start -1.524 0.762) (end -1.524 -0.762) (layer F.SilkS) (width 0.09906))
+    (fp_line (start -1.524 -0.762) (end -0.508 -0.762) (layer F.SilkS) (width 0.09906))
+    (fp_line (start 0.508 -0.762) (end 1.524 -0.762) (layer F.SilkS) (width 0.09906))
+    (fp_line (start 1.524 -0.762) (end 1.524 0.762) (layer F.SilkS) (width 0.09906))
+    (fp_line (start 1.524 0.762) (end 0.508 0.762) (layer F.SilkS) (width 0.09906))
+    (pad 1 smd rect (at -0.9525 0 270) (size 0.889 1.397)
+      (layers F.Cu F.Paste F.Mask)
+      (net 6 N-000004)
+    )
+    (pad 2 smd rect (at 0.9525 0 270) (size 0.889 1.397)
+      (layers F.Cu F.Paste F.Mask)
+      (net 2 /INJ-11)
+    )
+    (pad 2 thru_hole circle (at 1.905 0 270) (size 1.524 1.524) (drill 0.8128)
+      (layers *.Cu *.Mask F.SilkS)
+      (net 2 /INJ-11)
+    )
+    (pad 1 thru_hole circle (at -1.905 0 270) (size 1.524 1.524) (drill 0.8128)
+      (layers *.Cu *.Mask F.SilkS)
+      (net 6 N-000004)
+    )
+    (model smd/chip_cms.wrl
+      (at (xyz 0 0 0))
+      (scale (xyz 0.1 0.1 0.1))
+      (rotate (xyz 0 0 0))
+    )
+  )
+  (module SM0805_jumper (layer F.Cu)
+    (at 200.66 125.603 270)
+    (attr smd)
+    (fp_text reference W3 (at 0.0635 0 360) (layer F.SilkS)
+      (effects (font (size 0.762 0.762) (thickness 0.127)))
+    )
+    (fp_text value TEST (at 0 1.27 270) (layer F.SilkS) hide
+      (effects (font (size 0.50038 0.50038) (thickness 0.10922)))
+    )
+    (fp_circle (center -1.651 0.762) (end -1.651 0.635) (layer F.SilkS) (width 0.09906))
+    (fp_line (start -0.508 0.762) (end -1.524 0.762) (layer F.SilkS) (width 0.09906))
+    (fp_line (start -1.524 0.762) (end -1.524 -0.762) (layer F.SilkS) (width 0.09906))
+    (fp_line (start -1.524 -0.762) (end -0.508 -0.762) (layer F.SilkS) (width 0.09906))
+    (fp_line (start 0.508 -0.762) (end 1.524 -0.762) (layer F.SilkS) (width 0.09906))
+    (fp_line (start 1.524 -0.762) (end 1.524 0.762) (layer F.SilkS) (width 0.09906))
+    (fp_line (start 1.524 0.762) (end 0.508 0.762) (layer F.SilkS) (width 0.09906))
+    (pad 1 smd rect (at -0.9525 0 270) (size 0.889 1.397)
+      (layers F.Cu F.Paste F.Mask)
+      (net 4 N-000002)
+    )
+    (pad 2 smd rect (at 0.9525 0 270) (size 0.889 1.397)
+      (layers F.Cu F.Paste F.Mask)
+      (net 1 /INJ-10)
+    )
+    (pad 2 thru_hole circle (at 1.905 0 270) (size 1.524 1.524) (drill 0.8128)
+      (layers *.Cu *.Mask F.SilkS)
+      (net 1 /INJ-10)
+    )
+    (pad 1 thru_hole circle (at -1.905 0 270) (size 1.524 1.524) (drill 0.8128)
+      (layers *.Cu *.Mask F.SilkS)
+      (net 4 N-000002)
+    )
+    (model smd/chip_cms.wrl
+      (at (xyz 0 0 0))
+      (scale (xyz 0.1 0.1 0.1))
+      (rotate (xyz 0 0 0))
+    )
+  )
+  (module pin_array_8x2 (layer F.Cu)
+    (at 275.59 171.704 90)
+    (descr "Double rangee de contacts 2 x 8 pins")
+    (tags CONN)
+    (fp_text reference P_VOID3 (at 0 -3.302 90) (layer F.SilkS)
+      (effects (font (size 1.016 1.016) (thickness 0.2032)))
+    )
+    (fp_text value CONN_8 (at 0 3.302 90) (layer F.SilkS)
+      (effects (font (size 1.016 1.016) (thickness 0.2032)))
+    )
+    (fp_line (start -9.906 2.286) (end -9.906 -2.286) (layer F.SilkS) (width 0.3048))
+    (fp_line (start -9.906 -2.286) (end 9.906 -2.286) (layer F.SilkS) (width 0.3048))
+    (fp_line (start 9.906 -2.286) (end 9.906 2.286) (layer F.SilkS) (width 0.3048))
+    (fp_line (start 9.906 2.286) (end -9.906 2.286) (layer F.SilkS) (width 0.3048))
+    (pad 1 thru_hole rect (at -8.89 1.27 90) (size 1.524 1.524) (drill 1.016)
+      (layers *.Cu *.Mask F.SilkS)
+    )
+    (pad 2 thru_hole circle (at -8.89 -1.27 90) (size 1.524 1.524) (drill 1.016)
+      (layers *.Cu *.Mask F.SilkS)
+    )
+    (pad 3 thru_hole circle (at -6.35 1.27 90) (size 1.524 1.524) (drill 1.016)
+      (layers *.Cu *.Mask F.SilkS)
+    )
+    (pad 4 thru_hole circle (at -6.35 -1.27 90) (size 1.524 1.524) (drill 1.016)
+      (layers *.Cu *.Mask F.SilkS)
+    )
+    (pad 5 thru_hole circle (at -3.81 1.27 90) (size 1.524 1.524) (drill 1.016)
+      (layers *.Cu *.Mask F.SilkS)
+    )
+    (pad 6 thru_hole circle (at -3.81 -1.27 90) (size 1.524 1.524) (drill 1.016)
+      (layers *.Cu *.Mask F.SilkS)
+      (net 1 /INJ-10)
+    )
+    (pad 7 thru_hole circle (at -1.27 1.27 90) (size 1.524 1.524) (drill 1.016)
+      (layers *.Cu *.Mask F.SilkS)
+      (net 2 /INJ-11)
+    )
+    (pad 8 thru_hole circle (at -1.27 -1.27 90) (size 1.524 1.524) (drill 1.016)
+      (layers *.Cu *.Mask F.SilkS)
+      (net 3 /INJ-12)
+    )
+    (pad 9 thru_hole circle (at 1.27 1.27 90) (size 1.524 1.524) (drill 1.016)
+      (layers *.Cu *.Mask F.SilkS)
+    )
+    (pad 10 thru_hole circle (at 1.27 -1.27 90) (size 1.524 1.524) (drill 1.016)
+      (layers *.Cu *.Mask F.SilkS)
+    )
+    (pad 11 thru_hole circle (at 3.81 1.27 90) (size 1.524 1.524) (drill 1.016)
+      (layers *.Cu *.Mask F.SilkS)
+    )
+    (pad 12 thru_hole circle (at 3.81 -1.27 90) (size 1.524 1.524) (drill 1.016)
+      (layers *.Cu *.Mask F.SilkS)
+    )
+    (pad 13 thru_hole circle (at 6.35 1.27 90) (size 1.524 1.524) (drill 1.016)
+      (layers *.Cu *.Mask F.SilkS)
+    )
+    (pad 14 thru_hole circle (at 6.35 -1.27 90) (size 1.524 1.524) (drill 1.016)
+      (layers *.Cu *.Mask F.SilkS)
+    )
+    (pad 15 thru_hole circle (at 8.89 1.27 90) (size 1.524 1.524) (drill 1.016)
+      (layers *.Cu *.Mask F.SilkS)
+    )
+    (pad 16 thru_hole circle (at 8.89 -1.27 90) (size 1.524 1.524) (drill 1.016)
+      (layers *.Cu *.Mask F.SilkS)
+    )
+    (model pin_array/pins_array_8x2.wrl
+      (at (xyz 0 0 0))
+      (scale (xyz 1 1 1))
+      (rotate (xyz 0 0 0))
+    )
+  )
