File: hardware/frankenso_foundation/frankenso_foundation.kicad_pcb (KiCad board)
At the start: 2 copper layers, 154.1 x 161.7 mm, 66 parts, among them P99 176122-6_2ND

Commit message: making progress with the PCB
Parts:
- added P_VOID3: CONN_30, PIN_ARRAY_20X2, F.Cu at (287.7, -42.7)
- added P_VOID4: CONN_14, pin_array_8x2, F.Cu at (185.1, 242.8)
Connections:
- S1 pad 11: (no net) -> /HD44780_D4
- S1 pad 12: (no net) -> /HD44780_D5
- S1 pad 13: (no net) -> /HD44780_D6
- S1 pad 14: (no net) -> /HD44780_D7
- S1 pad 4: (no net) -> /HD44780_RS
- S1 pad 6: (no net) -> /HD44780_CS
- W39 pad 1: (no net) -> /INJ-GND
- W49 pad 1: (no net) -> /5V
- W50 pad 1: (no net) -> /INP2
- W51 pad 1: (no net) -> /3M
- W52 pad 1: (no net) -> /O2-SIG
- W53 pad 1: (no net) -> /INP1
- W54 pad 1: (no net) -> /IAT

Commit message: making progress with the PCB
Parts:
- added JP1: TEST, SM0805_jumper, F.Cu at (189.3, 143.1)
- added JP2: TEST, SIL-2, F.Cu at (127.0, 97.8)
- added JP3: TEST, SIL-2, F.Cu at (180.3, 97.8)
- added R99: 2K, SM0805, F.Cu at (196.8, 176.8)
- moved P_VOID4 92.8 mm to (148.9, 157.3), turned to 270 degrees
Connections:
- P_VOID3 pad 1: /INJ-GND -> GND
- P_VOID3 pad 10: (no net) -> /3J
- P_VOID3 pad 18: (no net) -> /3R
- P_VOID3 pad 2: (no net) -> /OUTPUT-GND
- P_VOID3 pad 3: (no net) -> /CPU-GND
- P_VOID3 pad 4: (no net) -> /INP11
- P_VOID3 pad 5: (no net) -> /CKP
- P_VOID3 pad 6: (no net) -> /3F
- P_VOID3 pad 7: (no net) -> /CID
- P_VOID3 pad 8: (no net) -> /3H
- P_VOID3 pad 9: (no net) -> /3I
- P_VOID4 pad 10: /GND -> GND
- P_VOID4 pad 12: (no net) -> GND
- P_VOID4 pad 13: (no net) -> /HD44780_VCC
- P_VOID4 pad 14: /GND -> GND
- S1 pad 1: /GND -> GND
- S1 pad 2: (no net) -> /HD44780_VCC
- S1 pad 3: (no net) -> N-00000120
- S1 pad 5: /GND -> GND
- S1 pad A: (no net) -> /HD44780_VCC
- S1 pad K: (no net) -> GND
- W1 pad 1: (no net) -> /12V-CONST
- W10 pad 1: (no net) -> /AC-RELAY
- W11 pad 1: (no net) -> /DIAG-1K
- W12 pad 1: (no net) -> /1L
- W13 pad 1: (no net) -> /1M
- W14 pad 1: (no net) -> /TPS-IDL-SW
- W15 pad 1: (no net) -> /STOP-LIGHT
- W16 pad 1: (no net) -> /STEERING-SW
- W17 pad 1: (no net) -> /AC-SW
- W18 pad 1: (no net) -> /COOL-FAN
- W19 pad 1: (no net) -> /BLOWER-SW
- W2 pad 1: (no net) -> /12V
- W20 pad 1: (no net) -> /REAR-DEFROSTER-SW
- W21 pad 1: (no net) -> /HEADLIGHT-SW
- W22 pad 1: (no net) -> /NEUTRAL-CLUTCH-SW
- W23 pad 1: (no net) -> /2A
- W24 pad 1: (no net) -> /2B
- W25 pad 1: (no net) -> /2C
- W26 pad 1: (no net) -> /2D
- W27 pad 1: (no net) -> /2E
- W28 pad 1: (no net) -> /2F
- W29 pad 1: (no net) -> /2G
- W3 pad 1: (no net) -> /START-SIG
- W30 pad 1: (no net) -> /2H
- W31 pad 1: (no net) -> /2I
- W32 pad 1: (no net) -> /2J
- W33 pad 1: (no net) -> /2K
- W34 pad 1: (no net) -> /2L
- W35 pad 1: (no net) -> /2M
- W36 pad 1: (no net) -> /2N
- W37 pad 1: (no net) -> /2O
- W38 pad 1: (no net) -> /2P
- W39 pad 1: /INJ-GND -> GND
- W4 pad 1: (no net) -> /DIAG
- W40 pad 1: (no net) -> /OUTPUT-GND
- W41 pad 1: (no net) -> /CPU-GND
- W42 pad 1: (no net) -> /INP11
- W43 pad 1: (no net) -> /CKP
- W44 pad 1: (no net) -> /3F
- W45 pad 1: (no net) -> /CID
- W46 pad 1: (no net) -> /3H
- W47 pad 1: (no net) -> /3I
- W48 pad 1: (no net) -> /3J
- W5 pad 1: (no net) -> /MUL
- W56 pad 1: (no net) -> /3R
- W6 pad 1: (no net) -> /1F
- W7 pad 1: (no net) -> /IGN
- W8 pad 1: (no net) -> /1H
- W9 pad 1: (no net) -> /1I

Commit message: making progress with the PCB
Parts:
- added P_VOID1: CONN_30, PIN_ARRAY_20X2, F.Cu at (139.1, 78.7)
- added P_VOID2: CONN_17, PIN_ARRAY_20X2, F.Cu at (191.1, 78.7)
- moved P_VOID3 129.4 mm to (243.2, 78.7)
Routing:
- net (no net): track 4.55 -> 0.00 mm
