File: trunk/hardware/rusefi_hardware_history/frankenso_rev00.40/frankenso/PWR_buck_12V_switcher.sch (KiCad schematic (older format))
At the start: 19 parts, among them P1002 CONN_1, P901 CONN_1, P902 CONN_1, Q1001 MOS_PRO, U1001 LM2596

Commit message: moving to 4.0
Parts:
- D1001: symbol ZENERSMALL -> ZENERsmall
- Q1001: symbol MOS_PRO -> MOS_Pro
Changed lines of the file:
@@
 EESchema Schematic File Version 2
+LIBS:frankenso-rescue
+LIBS:KICAD_Older_Version
 LIBS:power
 LIBS:device
@@
 LIBS:memory
 LIBS:xilinx
-LIBS:special
 LIBS:microcontrollers
 LIBS:dsp
@@
 LIBS:slc_oem
 LIBS:frankenso-cache
-EELAYER 27 0
+EELAYER 25 0
 EELAYER END
 $Descr A 11000 8500
@@
 $EndComp
 $Comp
-L MOS_PRO Q1001
+L MOS_Pro Q1001
 U 1 1 52C6272D
 P 4950 6500
@@
 $EndComp
 $Comp
-L ZENERSMALL D1001
+L ZENERsmall D1001
 U 1 1 533A08FB
 P 5250 6600
