File: trunk/hardware/rusefi_hardware_history/frankenso_rev00.40/frankenso/frankenso.sch (KiCad schematic (older format))
At the start: 107 parts, among them P10 CONN_1, P101 CONN_1, P11 CONN_1, P12 CONN_1, P13 CONN_1, P15 CONN_1, P16 CONN_1, P17 CONN_1, P18 CONN_1, P19 CONN_1, P20 CONN_1, P21 CONN_1, P22 CONN_1, P23 CONN_1, P30 CONN_1, P51 CONN_1, P52 CONN_1, P6 CONN_1, P9 CONN_1, P99 176122-6_2ND, U4 ITEAD_HC-0X, U5 SKRHAAE010

Commit message: moving to 4.0
Parts:
- P99: symbol 176122-6_2ND -> 176122-6_2nd
Changed lines of the file:
@@
 EESchema Schematic File Version 2
+LIBS:frankenso-rescue
+LIBS:KICAD_Older_Version
 LIBS:power
 LIBS:device
@@
 LIBS:memory
 LIBS:xilinx
-LIBS:special
 LIBS:microcontrollers
 LIBS:dsp
@@
 LIBS:slc_oem
 LIBS:frankenso-cache
-EELAYER 27 0
+EELAYER 25 0
 EELAYER END
 $Descr B 17000 11000
@@
 $EndComp
 $Comp
-L 176122-6_2ND P99
+L 176122-6_2nd P99
 U 1 1 5398DBFC
 P 5850 1200
@@
 $EndComp
 $Comp
-L 176122-6_2ND P99
+L 176122-6_2nd P99
 U 2 1 5398DC09
 P 8400 1200
@@
 $EndComp
 $Comp
-L 176122-6_2ND P99
+L 176122-6_2nd P99
 U 3 1 5398DC0F
 P 10900 1200
