File: trunk/hardware/rusefi_hardware_history/frankenso_rev00.40/frankenso/mmc_usb_1.sch (KiCad schematic (older format))
At the start: 28 parts, among them J351 MINI-USB-5P-3400020P1, J352 MINI-USB-5P-3400020P1V, P352 MICRO-SDCARD-CONNECTOR-330006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, Q701 MOS_PRO, U351 FT232RL

Commit message: moving to 4.0
Parts:
- Q701: symbol MOS_PRO -> MOS_Pro
Changed lines of the file:
@@
 EESchema Schematic File Version 2
+LIBS:frankenso-rescue
+LIBS:KICAD_Older_Version
 LIBS:power
 LIBS:device
@@
 LIBS:memory
 LIBS:xilinx
-LIBS:special
 LIBS:microcontrollers
 LIBS:dsp
@@
 LIBS:slc_oem
 LIBS:frankenso-cache
-EELAYER 27 0
+EELAYER 25 0
 EELAYER END
 $Descr A4 11693 8268
@@
 Connection ~ 3825 2300
 $Comp
-L MOS_PRO Q701
+L MOS_Pro Q701
 U 1 1 53E7E9F8
 P 8100 1575
